Commit message: Remove drone mesh dependancy

File: catkin_ws/src/dji_m600_sim/urdf/links.xacro (robot description, xacro)
@@ -17,10 +17,10 @@
     <link name="vehicle_center_link">
       <visual>
-        <geometry>
-          <mesh filename="file://$(find dji_m600_sim)/meshes/m600.dae" scale="${chassisScale} ${chassisScale} ${chassisScale}"/>
-        </geometry>
+        <!-- <geometry> -->
+          <!-- <mesh filename="file://$(find dji_m600_sim)/meshes/m600.dae" scale="${chassisScale} ${chassisScale} ${chassisScale}"/> -->
+        <!-- </geometry> -->
         <origin rpy="0 0 0" xyz="${chassisMeshXoffset} ${chassisMeshYoffset} ${chassisMeshZoffset}" />
-        <!-- <xacro:drone_cylinder /> -->
-        <!-- <material name="blue" /> -->
+        <xacro:drone_cylinder />
+        <material name="blue" />
       </visual>
       <collision>
